File: kicad/starbie.kicad_sch (KiCad schematic)
At the start: 0 parts

Commit message: update
Parts:
- added SW1: SW_Push, Button_Switch_THT:SW_NKK_GW12LJP, symbol Switch:SW_Push
- added U1: XIAO-ESP32-C3-SMD, Seeed_Studio_XIAO_Series:XIAO-ESP32-C3-SMD, symbol Seeed_Studio_XIAO_Series:XIAO-ESP32-C3-SMD
Connections:
- new net +3.3V: U1.12 (3V3_OUT)
- new net +5V: U1.14 (VBUS)
- new net GND: SW1.2, U1.13 (GND), U1.18 (GND)
- no-connect marks 0 -> 13
