File: kicad/_restore_backup_2026-10-07T12-23-06-875/starbie.kicad_sch (KiCad schematic)
At the start: 7 parts, among them J1 Conn_01x04_Pin, J2 Conn_01x08_Pin, SW1 SW_Push, SW2 SW_Push, U1 XIAO-ESP32-C3-SMD, U2 DHT11

Commit message: finished pcb :)
Parts:
- U1: footprint Imported parts:XIAO-ESP32-C3-SMD -> Imported parts:XIAO-ESP32-C6-DIP
Connections:
- net DHT11 DATA: no longer R1.2, U1.2 (D1), U2.2 (DATA)
- net GPIO2: no longer SW1.1, U1.3 (D2)
- net GPIO3: no longer SW2.1, U1.4 (D3)
- net SCA: no longer J1.4 (Pin_4)
- net SCL: no longer J1.3 (Pin_3), J2.3 (Pin_3), U1.5 (D4)
- net SDA: no longer J2.4 (Pin_4), U1.6 (D5)
Changed lines of the file:
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@@
 	)
 	(label "GPIO2"
-		(at 36.83 77.47 180)
+		(at 29.21 78.74 0)
 		(effects
 			(font
 				(size 1.27 1.27)
 			)
-			(justify right bottom)
+			(justify left bottom)
 		)
 	)
 	(label "SDA"
-		(at 175.26 106.68 0)
+		(at 176.53 107.95 0)
 		(effects
 			(font
@@
 	)
 	(label "DHT11 DATA"
-		(at 138.43 71.12 180)
+		(at 127 71.12 0)
 		(effects
 			(font
 				(size 1.27 1.27)
 			)
-			(justify right bottom)
+			(justify left bottom)
 		)
 	)
@@
 	)
 	(label "DHT11 DATA"
-		(at 133.35 48.26 0)
+		(at 134.62 48.26 0)
 		(effects
 			(font
@@
 	)
 	(label "SCA"
-		(at 179.07 48.26 270)
+		(at 180.34 53.34 90)
 		(effects
 			(font
 				(size 1.27 1.27)
 			)
-			(justify right bottom)
+			(justify left bottom)
 		)
 	)
@@
 	)
 	(label "GPIO3"
-		(at 123.19 113.03 180)
+		(at 116.84 114.3 0)
 		(effects
 			(font
 				(size 1.27 1.27)
 			)
-			(justify right bottom)
+			(justify left bottom)
 		)
 	)
 	(label "DHT11 DATA"
-		(at 36.83 73.66 180)
+		(at 24.13 74.93 0)
 		(effects
 			(font
 				(size 1.27 1.27)
 			)
-			(justify right bottom)
+			(justify left bottom)
 		)
 	)
@@
 	)
 	(label "SDA"
-		(at 36.83 88.9 180)
+		(at 31.75 90.17 0)
 		(effects
 			(font
 				(size 1.27 1.27)
 			)
-			(justify right bottom)
+			(justify left bottom)
 		)
 	)
 	(label "SCL"
-		(at 175.26 104.14 0)
+		(at 176.53 105.41 0)
 		(effects
 			(font
@@
 	)
 	(label "GPIO3"
-		(at 36.83 81.28 180)
+		(at 29.21 82.55 0)
 		(effects
 			(font
 				(size 1.27 1.27)
 			)
-			(justify right bottom)
+			(justify left bottom)
 		)
 	)
 	(label "SCL"
-		(at 36.83 85.09 180)
+		(at 31.75 86.36 0)
 		(effects
 			(font
 				(size 1.27 1.27)
 			)
-			(justify right bottom)
+			(justify left bottom)
 		)
 	)
@@
 	)
 	(label "SCL"
-		(at 176.53 48.26 270)
+		(at 177.8 53.34 90)
 		(effects
 			(font
 				(size 1.27 1.27)
 			)
-			(justify right bottom)
+			(justify left bottom)
 		)
 	)
 	(label "GPIO2"
-		(at 123.19 95.25 180)
+		(at 116.84 96.52 0)
 		(effects
 			(font
 				(size 1.27 1.27)
 			)
-			(justify right bottom)
+			(justify left bottom)
 		)
 	)
@@
 	)
 	(symbol
-		(lib_name "LOGO_1")
-		(lib_id "cat-bleh:LOGO")
-		(at 38.1 124.46 0)
-		(unit 1)
-		(body_style 1)
-		(exclude_from_sim no)
-		(in_bom yes)
-		(on_board yes)
-		(in_pos_files yes)
-		(dnp no)
-		(fields_autoplaced yes)
-		(property "Reference" "#G2"
-			(at 38.1 105.0971 0)
-			(hide yes)
-			(show_name no)
-			(do_not_autoplace no)
-			(effects
-				(font
-					(size 1.27 1.27)
-				)
-			)
-		)
-		(property "Value" "LOGO"
-			(at 38.1 143.8229 0)
-			(hide yes)
-			(show_name no)
-			(do_not_autoplace no)
-			(effects
-				(font
-					(size 1.27 1.27)
-				)
-			)
-		)
-		(property "Footprint" ""
-			(at 38.1 124.46 0)
-			(hide yes)
-			(show_name no)
-			(do_not_autoplace no)
-			(effects
-				(font
-					(size 1.27 1.27)
-				)
-			)
-		)
-		(property "Datasheet" ""
-			(at 38.1 124.46 0)
-			(hide yes)
-			(show_name no)
-			(do_not_autoplace no)
-			(effects
-				(font
-					(size 1.27 1.27)
-				)
-			)
-		)
-		(property "Description" ""
-			(at 38.1 124.46 0)
-			(hide yes)
-			(show_name no)
-			(do_not_autoplace no)
-			(effects
-				(font
-					(size 1.27 1.27)
-				)
-			)
-		)
-		(instances
-			(project "starbie"
-				(path "/7b0fa391-a9c3-41aa-9f87-65fbcdb77f46"
-					(reference "#G2")
-					(unit 1)
-				)
-			)
-		)
-	)
-	(symbol
 		(lib_id "power:+3.3V")
 		(at 184.15 54.61 0)
@@
 			)
 		)
-		(property "Footprint" "Imported parts:XIAO-ESP32-C3-SMD"
+		(property "Footprint" "Imported parts:XIAO-ESP32-C6-DIP"
 			(at 21.082 101.854 0)
 			(hide yes)
